File: kiCad_mk1/kiCad_mk1.kicad_sch (KiCad schematic)
At the start: 17 parts, among them J1 Barrel_Jack, J2 ToANGEL, J3 DCDC_BOOST, Q1 Q_NMOS_GDS, U2 ESP32-C6-DevKitC-1, X1 NeoPixel_Ring_1, X2 NeoPixel_Ring_2, X3 NeoPixel_Ring_3, X4 NeoPixel_Ring_4

Commit message: checkpoint
Parts:
- added BZ1: BZZLTR_MOLEDY_MAKER, symbol Device:Buzzer
- added SW1: ACTION1, symbol Switch:SW_Push_45deg
- added SW2: ACTION2, symbol Switch:SW_Push_45deg
- added SW3: ACTION3, symbol Switch:SW_Push_45deg
- added SW4: RotaryEncoder_Switch, symbol Device:RotaryEncoder_Switch
- added U1: AT42QT2120-MMHR, AT42QT2120-MMHR:QFN45P300X300X85-21N, symbol AT42QT2120-MMHR:AT42QT2120-MMHR
- D1: value LED_45deg -> FLARE
Connections:
- net GND is gone; now on net GNDPWR: C1.2, C2.2, C3.2, C4.2, J1.1, J2.1 (Pin_1), J3.1 (Pin_1), R3.2, U2.15 (GND), X1.1 (Pin_1), X2.1 (Pin_1), X3.1 (Pin_1), X4.1 (Pin_1)
- net at Q1.1 (G), R2.2: now also R3.1
- net at R1.2, U2.3 (GPIO4/MTMS): now also U2.1 (3V3), U2.2 (EN/RESET), U2.4 (GPIO5/MTDI), SW1.2
- net at U2.10 (GPIO10): now also SW2.2
- net at U2.11 (GPIO11): now also SW3.2
- net GNDPWR: now reaches U2.21 (GND)
- net GNDPWR: now also Q1.3 (S), BZ1.2 (-), SW1.1, SW2.1, SW3.1, SW4.C, SW4.S2
- net at U2.24 (GPIO19): now also SW4.A
- net at U2.25 (GPIO20): now also BZ1.1 (+)
- net at U2.26 (GPIO21): now also SW4.B
- net at U2.27 (GPIO22): now also SW4.S1
Other:
- moved on the sheet: C1, C2, C3, C4, D1, J1, J2, J3, Q1, R1, R2, R3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

Commit message: jazz
Parts:
- removed J2: ToANGEL, symbol Connector_Generic:Conn_01x02
- removed J3: DCDC_BOOST, symbol Connector_Generic:Conn_01x03
- removed U1: AT42QT2120-MMHR, AT42QT2120-MMHR:QFN45P300X300X85-21N, symbol AT42QT2120-MMHR:AT42QT2120-MMHR
- added D2, D3: 1N5819, symbol Device:D_Schottky
- added J3, J5: DCDC_BOOST, symbol Connector_Generic:Conn_01x04
- added J4: RADAR, symbol Connector_Generic:Conn_01x05
- added J6: ANGEL, symbol Connector_Generic:Conn_01x04
- added J7: MATRIX, symbol Connector_Generic:Conn_01x04
- added R4, R5: 10kΩ, symbol Device:R
- BZ1: value BZZLTR_MOLEDY_MAKER -> MELODY_MAKER
Connections:
- net +5V: now also J3.2 (Pin_2), J6.1 (Pin_1); no longer C2.1, J1.2
- net GNDPWR: now also J3.1 (Pin_1), J3.4 (Pin_4), J4.2 (Pin_2), J5.2 (Pin_2), J5.3 (Pin_3), J6.2 (Pin_2), J7.2 (Pin_2), R5.2
- net at U2.12 (GPIO2): now also J4.4 (Pin_4)
- net at U2.13 (GPIO3): now also J4.3 (Pin_3)
- net at U2.25 (GPIO20): now also J4.5 (Pin_5); no longer BZ1.1 (+)
- net at U2.28 (GPIO23): now also BZ1.1 (+)
- net at U2.29 (GPIO15/JTAG): now also J6.4 (Pin_4)
- net at U2.6 (GPIO7): now also J7.3 (Pin_3)
- net at U2.7 (GPIO0): now also J7.4 (Pin_4)
- net at U2.8 (GPIO1): now also R4.2, R5.1
- net at C3.1, D1.2 (A): now also J3.3 (Pin_3)
- new net: C2.1, D2.1 (K), D3.1 (K)
- new net: J5.1 (Pin_1), J6.3 (Pin_3)
- new net: D3.2 (A), J5.4 (Pin_4)
- new net: R1.2, U2.3 (GPIO4/MTMS)
- new net: D2.2 (A), J1.2, R4.1
- new net: J4.1 (Pin_1), J7.1 (Pin_1), U2.1 (3V3)
- new net: SW1.2, U2.4 (GPIO5/MTDI)
- now unconnected: U2.2 (EN/RESET)
Other:
- moved on the sheet: BZ1, C1, C2, C3, C4, D1, J1, Q1, R1, R2, R3, SW1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
